File: pcb/rev0/aqp_controller/aqp_controller.kicad_pcb (KiCad board)
At the start: 4 copper layers, 134.4 x 56 mm, 85 parts, among them J1 AMPHENOL_10118194-0001LF, J2 Conn_02x03_Odd_Even, J3 LD09S33E4GX00LF, J4 B2B-PH-K-S_LF__SN_, M1 COM-09032, Q1 L8050QLT1G, Q2 L8050QLT1G, Q3 DMG2301L, SW1 SW_Slide_DPDT, SW10 SW_Push, SW11 SW_Push, SW2 SW_Push, SW3 EG2219, SW4 SKRPACE010, SW5 SKRPACE010, SW6 SW_Push, SW7 SW_Push, SW8 SW_Push, SW9 SW_Push, U1 IP4234CZ6, U2 74HC595, U3 74HC595, U4 MCP73831-2-MC, U5 CP2102N-Axx-xQFN28, U6 AP7361C-33E, U7 ESP32-S3-WROOM-1-N16R8

Commit message: Big update, post CODE completion
Parts:
- removed the C1 at (87.9, 88.8)
- removed C13: 0.1u@50v, Capacitor_SMD:C_0402_1005Metric
- removed C16, C17: 1u@25v, Capacitor_SMD:C_0603_1608Metric
- removed the C2 at (95.4, 88.8)
- removed the C5 at (125.6, 88.3)
- removed the C7 at (124.0, 92.4)
- removed the C8 at (127.1, 100.6)
- removed D10, D11, D12, D5, D8, D9: D, Diode_SMD:D_0603_1608Metric
- removed the D2 at (198.3, 76.4)
- removed the D4 at (150.9, 83.0)
- removed the J2 at (87.6, 98.0)
- removed the Q1 at (127.1, 82.0)
- removed Q2: L8050QLT1G, Package_TO_SOT_SMD:SOT-23
- removed the R11 at (147.8, 79.8)
- removed R15: 1K, Resistor_SMD:R_0402_1005Metric
- removed R16, R17, R25, R29: 0, Resistor_SMD:R_0402_1005Metric
- removed R19, R24: 5K, Resistor_SMD:R_0402_1005Metric
- removed R21: 22K1, Resistor_SMD:R_0402_1005Metric
- removed R22: 47K5, Resistor_SMD:R_0402_1005Metric
- removed R23: 10K, Resistor_SMD:R_0402_1005Metric
- removed the R6 at (124.6, 81.1)
- removed the R7 at (124.6, 83.0)
- removed the R8 at (133.7, 81.0)
- removed the R9 at (133.7, 83.0)
- removed the SW4 at (124.0, 103.6)
- removed the SW5 at (148.0, 103.5)
- removed the U2 at (84.2, 88.6)
- removed the U3 at (91.7, 88.6)
- removed U5: CP2102N-Axx-xQFN28, Package_DFN_QFN:QFN-28-1EP_5x5mm_P0.5mm_EP3.35x3.35mm
- added J1: SolderJumper_2_Bridged, Jumper:SolderJumper-2_P1.3mm_Open_RoundedPad1.0x1.5mm, F.Cu at (104.2, 75.9)
- added J4: Conn_01x09, Connector_PinSocket_2.54mm:PinSocket_1x09_P2.54mm_Horizontal, B.Cu at (80.7, 85.6)
- C1: renamed from C10; value 4.7u@25v -> 4.7u@10v
- C2: renamed from C9; value 4.7u@25v -> 4.7u@10v
- C3: renamed from C6; value 10n@25v -> 10n@50v
- C4: renamed from C3; value 4.7u@25v -> 4.7u@10v
- C5: renamed from C4; value 4.7u@25v -> 4.7u@10v
- C6: renamed from C11; value 100n@25v -> 100n@50v
- C8: renamed from C14; value 10u@25v -> 22u@10v
- C9: renamed from C15; value 0.1u@50v -> 0.1u@16v
- J3: value LD09S33E4GX00LF -> Conn_01x03; footprint aqp_controller:AMPHENOL_LD09S33E4GX00LF -> Connector_PinHeader_2.54mm:PinHeader_1x03_P2.54mm_Vertical; moved to F.Cu
- R1: renamed from R3; value 5K -> 1K
- R11: renamed from R12; value 5K -> 1K
- R3: renamed from R4; value 5K -> 1K
- R4: renamed from R5; value 5K -> 1K
- R5: renamed from R2; value 5K -> 1K
- R6: renamed from R20; value 5K -> 1K
- R8: renamed from R1; value 5K -> 1K
- R9: renamed from R13; value 5K -> 1K
- SW1: value SW_Slide_DPDT -> SKRPACE010; footprint Button_Switch_THT:SW_CK_JS202011AQN_DPDT_Angled -> aqp_controller:SW_SKRPACE010
- moved C2 54.6 mm to (132.7, 83.4), turned to 90 degrees
- moved C1 51.3 mm to (123.2, 83.4), turned to 90 degrees
- moved U2 48.6 mm to (127.9, 86.3), turned to -90 degrees
- moved SW1 36.2 mm to (95.3, 76.5)
- moved J3 31.8 mm to (122.3, 108.0)
- moved R11 23.0 mm to (85.3, 105.9), turned to 180 degrees
- moved R8 21.2 mm to (85.3, 100.8)
- moved R9 20.0 mm to (85.3, 103.4), turned to 180 degrees
- moved D4 19.9 mm to (131.2, 97.7), turned to -90 degrees
- moved R5 17.8 mm to (85.3, 98.3)
- moved R7 17.2 mm to (132.8, 96.9), turned to -90 degrees
- moved R10 16.5 mm to (125.0, 99.4), turned to 180 degrees
- moved U3 14.2 mm to (127.7, 97.1)
- moved C4 14.2 mm to (124.8, 97.2)
- moved C5 13.8 mm to (127.7, 99.3), turned to 0 degrees
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- renumbered C12 to C7, D3 to D1, D6 to D2, D7 to D3, D1 to D4, J1 to J2, J4 to J5, Q3 to Q1, R14 to R10, R27 to R12, R26 to R13, R28 to R14, R18 to R2, R10 to R7, SW3 to SW2, SW8 to SW3, SW2 to SW4, SW7 to SW5, SW11 to SW6, SW10 to SW7, SW6 to SW8, U6 to U2, U4 to U3, U7 to U4
Connections:
- C2 pad 2: Net-(D7-K) -> Net-(D3-K)
- C4 pad 2: Net-(D1-K) -> BATT+
- C7 pad 2: CHIP_PU -> ~{RESET}
- D1 pad 3: Net-(D3-DIN) -> RGBPIN
- D3 pad 1: Net-(D7-K) -> Net-(D3-K)
- D4 pad 1: Net-(D1-K) -> Net-(D4-K)
- J3 pad 1: D8 -> GND
- J3 pad 2: D7 -> U0RXD
- J3 pad 3: D6 -> U0TXD
- J5 pad 1: BATT- -> GND
- L1 pad 1: Net-(L1-Pad1) -> USB_DN
- L1 pad 4: Net-(L1-Pad4) -> USB_DP
- M1 pad B1A: COL1 -> BUTTONPIN_T
- M1 pad B2A: TH_SW- -> GND
- M1 pad H2: TH_X -> XPIN
- M1 pad V2: TH_Y -> YPIN
- Q1 pad 2: Net-(Q3-S) -> Net-(D3-K)
- Q1 pad 3: Net-(D7-K) -> SW_BATT+
- R1 pad 1: D5 -> DATAPIN_0
- R1 pad 2: PULLER -> D0
- R11 pad 1: D1 -> DATAPIN_7
- R11 pad 2: PULLER -> D7
- R13 pad 1: Net-(D7-K) -> Net-(D3-K)
- R14 pad 1: ESP_3V3 -> VCC_3V3
- R14 pad 2: CHIP_PU -> ~{RESET}
- R3 pad 1: D6 -> DATAPIN_1
- R3 pad 2: PULLER -> D1
- R4 pad 1: D7 -> DATAPIN_2
- R4 pad 2: PULLER -> D2
- R5 pad 1: D4 -> DATAPIN_4
- R5 pad 2: PULLER -> D4
- R6 pad 1: D0 -> DATAPIN_3
- R6 pad 2: PULLER -> D3
- R8 pad 1: D3 -> DATAPIN_5
- R8 pad 2: PULLER -> D5
- R9 pad 1: D2 -> DATAPIN_6
- R9 pad 2: PULLER -> D6
- SW1 pad 1: UART_DP -> ~{RESET}
- SW1 pad 2: Net-(L1-Pad4) -> unconnected-(SW1-Pad2)
- SW1 pad 3: USB_DP -> GND
- SW1 pad 4: USB_DN -> unconnected-(SW1-Pad4)
- SW2 pad 2: Net-(Q3-S) -> SW_BATT+
- SW2 pad 3: BATT- -> GND
- SW2 pad 5: Net-(Q3-S) -> SW_BATT+
- SW2 pad 6: BATT- -> GND
- SW2 pad S1: BATT- -> GND
- SW2 pad S2: BATT- -> GND
- SW2 pad S3: BATT- -> GND
- SW2 pad S4: BATT- -> GND
- SW3 pad 1: COL2 -> BUTTONPIN_6
- SW3 pad 3: Net-(D2-A) -> GND
- SW4 pad 1: COL0 -> BUTTONPIN_G
- SW4 pad 3: Net-(D4-A) (its old number) -> GND
- SW5 pad 1: COL1 -> BUTTONPIN_5
- SW5 pad 3: Net-(D5-A) -> GND
- SW6 pad 1: COL2 -> BUTTONPIN_3
- SW6 pad 3: Net-(D9-A) -> GND
- SW7 pad 1: COL1 -> BUTTONPIN_2
- SW7 pad 3: Net-(D10-A) -> GND
- SW8 pad 1: COL0 -> BUTTONPIN_4
- SW8 pad 3: Net-(D8-A) -> GND
- SW9 pad 1: COL0 -> BUTTONPIN_1
- SW9 pad 3: Net-(D11-A) -> GND
- U2 pad 1: Net-(D7-K) -> Net-(D3-K)
- U3 pad 5: Net-(D1-K) -> Net-(D4-K)
- U4 pad 10: COL1 -> DATAPIN_7
- U4 pad 11: COL2 -> DATAPIN_3
- U4 pad 12: GPIO8 -> BUTTONPIN_4
- U4 pad 15: GPIO3 -> unconnected-(U4-IO3-Pad15)
- U4 pad 16: SR_LATCH -> unconnected-(U4-IO46-Pad16)
- U4 pad 17: GPIO9 -> BUTTONPIN_5
- U4 pad 18: GPIO10 -> BUTTONPIN_6
- U4 pad 19: GPIO11 -> BUTTONPIN_G
- U4 pad 2: ESP_3V3 -> VCC_3V3
- U4 pad 20: GPIO12 -> unconnected-(U4-IO12-Pad20)
- U4 pad 21: GPIO13 -> BATDIV
- U4 pad 22: SR_DATA -> unconnected-(U4-IO14-Pad22)
- U4 pad 23: SR_CLK -> DATAPIN_2
- U4 pad 24: TH_Y -> unconnected-(U4-IO47-Pad24)
- U4 pad 25: LED_DATA -> RGBPIN
- U4 pad 26: TH_X -> unconnected-(U4-IO45-Pad26)
- U4 pad 27: AUTO_PRG -> BOOTLOADER
- U4 pad 28: GPIO35 -> unconnected-(U4-IO35-Pad28)
- U4 pad 29: GPIO36 -> unconnected-(U4-IO36-Pad29)
- U4 pad 3: CHIP_PU -> ~{RESET}
- U4 pad 30: GPIO37 -> unconnected-(U4-IO37-Pad30)
- U4 pad 31: GPIO38 -> DATAPIN_1
- U4 pad 32: GPIO39 -> DATAPIN_0
- U4 pad 33: GPIO40 -> DATAPIN_4
- U4 pad 34: GPIO41 -> DATAPIN_5
- U4 pad 35: BATDIV -> DATAPIN_6
- U4 pad 38: GPIO2 -> unconnected-(U4-IO2-Pad38)
- U4 pad 39: GPIO1 -> unconnected-(U4-IO1-Pad39)
- U4 pad 4: GPIO4 -> BUTTONPIN_T
- U4 pad 5: GPIO5 -> BUTTONPIN_1
- U4 pad 6: ROW0 -> BUTTONPIN_2
- U4 pad 7: ROW1 -> BUTTONPIN_3
- U4 pad 8: ROW2 -> XPIN
- U4 pad 9: COL0 -> YPIN
Routing:
- net BATT-: track 131.8 -> 0.00 mm, vias 4 -> 0
- net VCC_3V3: track 232.3 -> 110.8 mm, vias 10 -> 2
- net COL1: track 105.2 -> 0.00 mm, vias 2 -> 0
- net Net-(D7-K): track 98.2 -> 0.00 mm, vias 4 -> 0
- net ~{RESET}: track 0.00 -> 86.8 mm, vias 0 -> 4
- net Net-(D3-K): track 0.00 -> 77.6 mm, vias 0 -> 2
- net COL2: track 75.0 -> 0.00 mm, vias 1 -> 0
- net DATAPIN_3: track 0.00 -> 74.9 mm, vias 0 -> 4
- net COL0: track 73.8 -> 0.00 mm, vias 2 -> 0
- net ROW0: track 73.6 -> 0.00 mm, vias 4 -> 0
- net BUTTONPIN_6: track 0.00 -> 72.3 mm, vias 0 -> 2
- net ROW2: track 69.9 -> 0.00 mm, vias 5 -> 0
- net SR_LATCH: track 68.6 -> 0.00 mm, vias 3 -> 0
- net ROW1: track 68.6 -> 0.00 mm, vias 2 -> 0
- net XPIN: track 0.00 -> 67.3 mm, vias 0 -> 2
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- removed copper zone on In1.Cu, net GND
- removed copper zone on In2.Cu, net VCC_3V3
Other:
- copper layers 4 -> 2
- board text added: "20241204"
- board text added: "Battery Mgmt"
- board text added: "D0"
- board text added: "D1"
- board text added: "D2"
- board text added: "D3"
- board text added: "D4"
- board text added: "D5"
- board text added: "D6"
- board text added: "D7"
- board text added: "DEBUG"
- board text added: "DP1"
- board text added: "DP2"
- board text added: "DP3"
- board text added: "DP4"
- board text added: "DP5"
- board text added: "DP6"
- board text added: "DP7"
- board text added: "DP8"
- board text added: "DP9"
- board text added: "Gamepad"
- board text added: "Rx"
- board text added: "Tx"
- board text removed: "+3.3V"
- board text removed: "+5V"
- board text removed: "1"
- board text removed: "2"
- board text removed: "20241106"
- board text removed: "3"
- board text removed: "4"
- board text removed: "5"
- board text removed: "6"
- board text removed: "7"
- board text removed: "8"
- board text removed: "9"
- board text removed: "Batt"
- board text removed: "Common"
- board text removed: "Game Controller"
- board text removed: "Mgmt"
- board text removed: "Shift Regs"
- board text removed: "UART"
- board text removed: "USB"
