File: pcb/rev0/aqp_controller/aqp_controller.kicad_sch (KiCad schematic)
At the start: 85 parts, among them J1 AMPHENOL_10118194-0001LF, J2 Conn_02x03_Odd_Even, J3 LD09S33E4GX00LF, J4 B2B-PH-K-S_LF__SN_, M1 COM-09032, Q1 L8050QLT1G, Q2 L8050QLT1G, Q3 DMG2301L, SW1 SW_Slide_DPDT, SW10 SW_Push, SW11 SW_Push, SW2 SW_Push, SW3 EG2219, SW4 SKRPACE010, SW5 SKRPACE010, SW6 SW_Push, SW7 SW_Push, SW8 SW_Push, SW9 SW_Push, U1 IP4234CZ6, U2 74HC595, U3 74HC595, U4 MCP73831-2-MC, U5 CP2102N-Axx-xQFN28, U6 AP7361C-33E, U7 ESP32-S3-WROOM-1-N16R8

Commit message: Big update, post CODE completion
Parts:
- removed C1, C2: 0.1u@25v, Capacitor_SMD:C_0603_1608Metric, symbol Device:C
- removed C13, C8: 0.1u@50v, Capacitor_SMD:C_0402_1005Metric, symbol Device:C
- removed C16, C17: 1u@25v, Capacitor_SMD:C_0603_1608Metric, symbol Device:C
- removed C5: 10u@25v, Capacitor_SMD:C_0603_1608Metric, symbol Device:C
- removed C7: 1u@16v, Capacitor_SMD:C_0402_1005Metric, symbol Device:C
- removed D10, D11, D12, D2, D4, D5, D8, D9: D, Diode_SMD:D_0603_1608Metric, symbol Device:D
- removed J2: Conn_02x03_Odd_Even, Connector_PinHeader_2.54mm:PinHeader_2x03_P2.54mm_Vertical, symbol Connector_Generic:Conn_02x03_Odd_Even
- removed J3: LD09S33E4GX00LF, aqp_controller:AMPHENOL_LD09S33E4GX00LF, symbol LD09S33E4GX00LF:LD09S33E4GX00LF
- removed Q1, Q2: L8050QLT1G, Package_TO_SOT_SMD:SOT-23, symbol Transistor_BJT:BC818
- removed R11, R16, R17, R25, R29, R6, R9: 0, Resistor_SMD:R_0402_1005Metric, symbol Device:R_US
- removed R15: 1K, Resistor_SMD:R_0402_1005Metric, symbol Device:R_US
- removed R19, R24: 5K, Resistor_SMD:R_0402_1005Metric, symbol Device:R_US
- removed R21: 22K1, Resistor_SMD:R_0402_1005Metric, symbol Device:R_US
- removed R22: 47K5, Resistor_SMD:R_0402_1005Metric, symbol Device:R_US
- removed R23, R7, R8: 10K, Resistor_SMD:R_0402_1005Metric, symbol Device:R_US
- removed SW1: SW_Slide_DPDT, Button_Switch_THT:SW_CK_JS202011AQN_DPDT_Angled, symbol Switch:SW_Slide_DPDT
- removed SW4, SW5: SKRPACE010, aqp_controller:SW_SKRPACE010, symbol SKRPACE010:SKRPACE010
- removed U2, U3: 74HC595, Package_SO:TSSOP-16_4.4x5mm_P0.65mm, symbol 74xx:74HC595
- removed U5: CP2102N-Axx-xQFN28, Package_DFN_QFN:QFN-28-1EP_5x5mm_P0.5mm_EP3.35x3.35mm, symbol Interface_USB:CP2102N-Axx-xQFN28
- added J1: SolderJumper_2_Bridged, Jumper:SolderJumper-2_P1.3mm_Open_RoundedPad1.0x1.5mm, symbol Jumper:SolderJumper_2_Bridged
- added J3: Conn_01x03, Connector_PinHeader_2.54mm:PinHeader_1x03_P2.54mm_Vertical, symbol Connector_Generic:Conn_01x03
- added J4: Conn_01x09, Connector_PinSocket_2.54mm:PinSocket_1x09_P2.54mm_Horizontal, symbol Connector_Generic:Conn_01x09
- added SW1: SKRPACE010, aqp_controller:SW_SKRPACE010, symbol SKRPACE010:SKRPACE010
- C1: renamed from C10; value 4.7u@25v -> 4.7u@10v; JLCPCB Part # C96446 -> C1705
- C2: renamed from C9; value 4.7u@25v -> 4.7u@10v; JLCPCB Part # C96446 -> C1705
- C3: renamed from C6; value 10n@25v -> 10n@50v; JLCPCB Part # C96446 -> C376807
- C4: renamed from C3; value 4.7u@25v -> 4.7u@10v; JLCPCB Part # C96446 -> C1705
- C5: renamed from C4; value 4.7u@25v -> 4.7u@10v; JLCPCB Part # C96446 -> C1705
- C6: renamed from C11; value 100n@25v -> 100n@50v; JLCPCB Part # C96446 -> C282519
- C8: renamed from C14; value 10u@25v -> 22u@10v; JLCPCB Part # C96446 -> C86295
- C9: renamed from C15; value 0.1u@50v -> 0.1u@16v; JLCPCB Part # C1581 -> C60474
- D2: renamed from D6; JLCPCB Part # (none) -> C552798
- D3: renamed from D7; JLCPCB Part # (none) -> C552798
- D4: renamed from D1; JLCPCB Part # C2297 -> C6795835
- J5: renamed from J4; now not fitted; now left out of the parts list
- L1: JLCPCB Part # (none) -> C2649327
- M1, SW9: now not fitted; now left out of the parts list
- Q1: renamed from Q3; JLCPCB Part # (none) -> C102619
- R1: renamed from R3; value 5K -> 1K; JLCPCB Part # C60485 -> C25543
- R10: renamed from R14; JLCPCB Part # C25744 -> C25933
- R11: renamed from R12; value 5K -> 1K; JLCPCB Part # C60485 -> C25543
- R12: renamed from R27; JLCPCB Part # C25905 -> C102750
- R13: renamed from R26; JLCPCB Part # C25905 -> C102750
- R14: renamed from R28; JLCPCB Part # C25744 -> C2906861
- R2: renamed from R18; JLCPCB Part # C25905 -> C102750
- R3: renamed from R4; value 5K -> 1K; JLCPCB Part # C60485 -> C25543
- R4: renamed from R5; value 5K -> 1K; JLCPCB Part # C60485 -> C25543
- R5: renamed from R2; value 5K -> 1K; JLCPCB Part # C60485 -> C25543
- R6: renamed from R20; value 5K -> 1K; JLCPCB Part # C60485 -> C25543
- R7: renamed from R10; JLCPCB Part # C25905 -> C25117
- R8: renamed from R1; value 5K -> 1K; JLCPCB Part # C60485 -> C25543
- R9: renamed from R13; value 5K -> 1K; JLCPCB Part # C60485 -> C25543
- SW2: renamed from SW3; now not fitted; now left out of the parts list
- SW3: renamed from SW8; now not fitted; now left out of the parts list
- SW4: renamed from SW2; now not fitted; now left out of the parts list
- SW5: renamed from SW7; now not fitted; now left out of the parts list
- SW6: renamed from SW11; now not fitted; now left out of the parts list
- SW7: renamed from SW10; now not fitted; now left out of the parts list
- SW8: renamed from SW6; now not fitted; now left out of the parts list
- U1: JLCPCB Part # (none) -> C455086
- U2: renamed from U6; JLCPCB Part # (none) -> C500795
- U3: renamed from U4; JLCPCB Part # (none) -> C635037
- U4: renamed from U7; JLCPCB Alt Part # C19170935 -> (none)
- renumbered C12 to C7, D3 to D1, J1 to J2
Connections:
- net BATT- is gone; now on net GND: J5.1, SW2.3, SW2.6, SW2.S1 (SHIELD), SW2.S2 (SHIELD__1), SW2.S3 (SHIELD__2), SW2.S4 (SHIELD__3)
- net ESP_3V3 is gone; now on net VCC_3V3: R14.1, U4.2 (3V3)
- net GPIO13 is gone; now on net BATDIV: U4.21 (IO13)
- net LED_DATA is gone; now on net RGBPIN: U4.25 (IO48)
- net TH_SW- is gone; now on net GND: M1.B2A (SEL-)
- net BATDIV: no longer U4.35 (IO42)
- net BATT+: now also C4.2
- net D0: now also R1.2, J4.2 (Pin_2); no longer R6.1
- net D1: now also R3.2, J4.3 (Pin_3); no longer R11.1
- net D2: now also R4.2, J4.4 (Pin_4); no longer R9.1
- net D3: now also R6.2, J4.5 (Pin_5); no longer R8.1
- net D4: now also R5.2, J4.6 (Pin_6); no longer R5.1
- net D5: now also R8.2, J4.7 (Pin_7); no longer R1.1
- net D6: now also R9.2, J4.8 (Pin_8); no longer R3.1
- net D7: now also R11.2, J4.9 (Pin_9); no longer R4.1
- net GND: now also SW3.3, SW4.3, SW5.3, SW6.3, SW7.3, SW8.3, SW9.3, J1.2 (B), J3.1 (Pin_1), J4.1 (Pin_1), SW1.3
- net U0RXD: now also J3.2 (Pin_2)
- net U0TXD: now also J3.3 (Pin_3)
- net USB_DN: now also L1.1
- net USB_DP: now also L1.4
- net SW_BATT+: now reaches SW2.2, SW2.5
- net SW_BATT+: now also Q1.3 (D); no longer Q1.2 (S)
- net at D4.1 (K), U3.5 (STAT): no longer C4.2
- net RGBPIN: now reaches D1.3 (DIN)
- net at C2.2, D3.1 (K), R13.1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: now also Q1.2 (S); no longer Q1.3 (D)
- net AUTO_PRG renamed BOOTLOADER
- net BOOTLOADER: now also J1.1 (A)
- net CHIP_PU renamed ~{RESET}
- net ~{RESET}: now also SW1.1
- removed net COL0: SW4.1, SW8.1, SW9.1, U4.9 (IO16)
- removed net COL1: M1.B1A (SEL+), SW5.1, SW7.1, U4.10 (IO17)
- removed net COL2: SW3.1, SW6.1, U4.11 (IO18)
- net GPIO1: no longer names the net of U4.39 (IO1)
- net GPIO10 renamed BUTTONPIN_6
- net BUTTONPIN_6: now also SW3.1
- net GPIO11 renamed BUTTONPIN_G
- net BUTTONPIN_G: now also SW4.1
- net GPIO12: no longer names the net of U4.20 (IO12)
- net GPIO2: no longer names the net of U4.38 (IO2)
- net GPIO3: no longer names the net of U4.15 (IO3)
- net GPIO35: no longer names the net of U4.28 (IO35)
- net GPIO36: no longer names the net of U4.29 (IO36)
- net GPIO37: no longer names the net of U4.30 (IO37)
- net GPIO38 renamed DATAPIN_1
- net DATAPIN_1: now also R3.1
- net GPIO39 renamed DATAPIN_0
- net DATAPIN_0: now also R1.1
- net GPIO4 renamed BUTTONPIN_T
- net BUTTONPIN_T: now also M1.B1A (SEL+)
- net GPIO40 renamed DATAPIN_4
- net DATAPIN_4: now also R5.1
- net GPIO41 renamed DATAPIN_5
- net DATAPIN_5: now also R8.1
- net GPIO5 renamed BUTTONPIN_1
- net BUTTONPIN_1: now also SW9.1
- net GPIO8 renamed BUTTONPIN_4
- net BUTTONPIN_4: now also SW8.1
- net GPIO9 renamed BUTTONPIN_5
- net BUTTONPIN_5: now also SW5.1
- removed net PULLER: R1.2, R11.2, R3.2, R4.2, R5.2, R6.2, R8.2, R9.2
- net ROW0 renamed BUTTONPIN_2
- net BUTTONPIN_2: now also SW7.1
- net ROW1 renamed BUTTONPIN_3
- net BUTTONPIN_3: now also SW6.1
- net ROW2 renamed XPIN
- net XPIN: now also M1.H2 (H)
- net SR_CLK renamed DATAPIN_2
- net DATAPIN_2: now also R4.1
- net SR_DATA: no longer names the net of U4.22 (IO14)
- net SR_LATCH: no longer names the net of U4.16 (IO46)
- net TH_X: no longer names the net of U4.26 (IO45)
- net TH_X: no longer M1.H2 (H)
- net TH_Y: no longer names the net of U4.24 (IO47)
- net TH_Y: no longer M1.V2 (V)
- new net DATAPIN_3: R6.1, U4.11 (IO18)
- new net DATAPIN_6: R9.1, U4.35 (IO42)
- new net DATAPIN_7: R11.1, U4.10 (IO17)
- new net YPIN: M1.V2 (V), U4.9 (IO16)
- no-connect marks 47 -> 29
Other:
- note added: "Battery"
- note added: "Boot"
- note added: "Buttons"
- note added: "Debug"
- note added: "ESP32"
- note added: "Power Management"
- note added: "RGB LED"
- note added: "Reset"
- note added: "Thumbstick"
- note added: "USB Port"
- note added: "Wired Interface"
- company: Aquarius+ -> Drawing by Sean P. Harrington
- title: Aquarius+ Controller -> Aquarius+ Gamepad
- moved on the sheet: C1, C2, C3, C4, C5, C6, C7, C8, C9, D1, D2, D3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
